File: project/makerspace_sign.kicad_pcb (KiCad board)
At the start: 2 copper layers, 76.2 x 98 mm, 23 parts, among them J1 Conn_EXT, J2 Conn_E1_M, J3 Conn_E1_F, J4 Conn_OTH_M, J5 Conn_OTH_F, J6 Conn_E2_F, J7 Conn_E2_M

Commit message: v1
Routing:
- net +12V: track 198.8 -> 200.2 mm
- net GND: vias 17 -> 19
Changed lines of the file:
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@@
   (via (at 77.2 95.5) (size 1.2) (drill 0.4) (layers "F.Cu" "B.Cu") (net 2))
   (via (at 102.6 86) (size 1.2) (drill 0.4) (layers "F.Cu" "B.Cu") (free) (net 2))
+  (via (at 134.6 94) (size 1.2) (drill 0.4) (layers "F.Cu" "B.Cu") (free) (net 2))
   (via (at 63.3 88.6) (size 1.2) (drill 0.4) (layers "F.Cu" "B.Cu") (free) (net 2))
   (via (at 118.1 110.5) (size 1.2) (drill 0.4) (layers "F.Cu" "B.Cu") (free) (net 2))
   (via (at 102.6 94.2) (size 1.2) (drill 0.4) (layers "F.Cu" "B.Cu") (free) (net 2))
   (via (at 117.1 88.1) (size 1.2) (drill 0.4) (layers "F.Cu" "B.Cu") (free) (net 2))
+  (via (at 64 69) (size 1.2) (drill 0.4) (layers "F.Cu" "B.Cu") (free) (net 2))
   (segment (start 92.755 97.555) (end 105.345 97.555) (width 0.6) (layer "F.Cu") (net 3))
   (segment (start 105.455 97.555) (end 108 97.555) (width 0.6) (layer "F.Cu") (net 3))
@@
   (via (at 126 87.2) (size 1.2) (drill 0.4) (layers "F.Cu" "B.Cu") (net 3))
   (via (at 125.9 103.5) (size 1.2) (drill 0.4) (layers "F.Cu" "B.Cu") (net 3))
+  (segment (start 90.4 67.1) (end 90.4 65.6) (width 0.6) (layer "B.Cu") (net 3))
+  (segment (start 126 87.2) (end 126 85.5) (width 0.6) (layer "B.Cu") (net 3))
+  (segment (start 96.9 120.3) (end 100.5 120.3) (width 0.6) (layer "B.Cu") (net 3))
+  (segment (start 125.9 105) (end 125.9 103.5) (width 0.6) (layer "B.Cu") (net 3))
   (segment (start 111.7 112) (end 113.4 112) (width 0.6) (layer "B.Cu") (net 3))
-  (segment (start 121.2 108.5) (end 125.9 103.8) (width 0.6) (layer "B.Cu") (net 3))
   (segment (start 100.5 120.3) (end 105.1 115.7) (width 0.6) (layer "B.Cu") (net 3))
-  (segment (start 122.1 83.2) (end 114.9 83.2) (width 0.6) (layer "B.Cu") (net 3))
-  (segment (start 95.6 120.3) (end 100.5 120.3) (width 0.6) (layer "B.Cu") (net 3))
+  (segment (start 96 72.7) (end 90.4 67.1) (width 0.6) (layer "B.Cu") (net 3))
+  (segment (start 122.4 108.5) (end 125.9 105) (width 0.6) (layer "B.Cu") (net 3))
+  (segment (start 88.5 63.7) (end 85.3 63.7) (width 0.6) (layer "B.Cu") (net 3))
   (segment (start 104.4 72.7) (end 96 72.7) (width 0.6) (layer "B.Cu") (net 3))
-  (segment (start 96 72.7) (end 90.4 67.1) (width 0.6) (layer "B.Cu") (net 3))
-  (segment (start 108 115.7) (end 111.7 112) (width 0.6) (layer "B.Cu") (net 3))
-  (segment (start 126 87.1) (end 122.1 83.2) (width 0.6) (layer "B.Cu") (net 3))
   (segment (start 83.4 126) (end 84.6 127.2) (width 0.6) (layer "B.Cu") (net 3))
   (segment (start 113.4 112) (end 116.9 108.5) (width 0.6) (layer "B.Cu") (net 3))
-  (segment (start 88.7 127.2) (end 95.6 120.3) (width 0.6) (layer "B.Cu") (net 3))
-  (segment (start 90.4 65.2) (end 88.3 63.1) (width 0.6) (layer "B.Cu") (net 3))
   (segment (start 126 103.4) (end 126 87.2) (width 0.6) (layer "B.Cu") (net 3))
-  (segment (start 116.9 108.5) (end 121.2 108.5) (width 0.6) (layer "B.Cu") (net 3))
-  (segment (start 84.6 127.2) (end 88.7 127.2) (width 0.6) (layer "B.Cu") (net 3))
+  (segment (start 105.1 115.7) (end 108 115.7) (width 0.6) (layer "B.Cu") (net 3))
+  (segment (start 90.4 65.6) (end 88.5 63.7) (width 0.6) (layer "B.Cu") (net 3))
+  (segment (start 108 115.7) (end 111.7 112) (width 0.6) (layer "B.Cu") (net 3))
+  (segment (start 113.5 81.8) (end 104.4 72.7) (width 0.6) (layer "B.Cu") (net 3))
   (segment (start 105.4 97.5) (end 83.4 119.5) (width 0.6) (layer "B.Cu") (net 3))
+  (segment (start 126 85.5) (end 122.3 81.8) (width 0.6) (layer "B.Cu") (net 3))
+  (segment (start 85.3 63.7) (end 84.7 63.1) (width 0.6) (layer "B.Cu") (net 3))
   (segment (start 125.9 103.5) (end 126 103.4) (width 0.6) (layer "B.Cu") (net 3))
-  (segment (start 105.1 115.7) (end 108 115.7) (width 0.6) (layer "B.Cu") (net 3))
-  (segment (start 90.4 67.1) (end 90.4 65.2) (width 0.6) (layer "B.Cu") (net 3))
-  (segment (start 114.9 83.2) (end 104.4 72.7) (width 0.6) (layer "B.Cu") (net 3))
+  (segment (start 116.9 108.5) (end 122.4 108.5) (width 0.6) (layer "B.Cu") (net 3))
+  (segment (start 90 127.2) (end 96.9 120.3) (width 0.6) (layer "B.Cu") (net 3))
+  (segment (start 122.3 81.8) (end 113.5 81.8) (width 0.6) (layer "B.Cu") (net 3))
   (segment (start 83.4 119.5) (end 83.4 126) (width 0.6) (layer "B.Cu") (net 3))
-  (segment (start 88.3 63.1) (end 84.7 63.1) (width 0.6) (layer "B.Cu") (net 3))
-  (segment (start 125.9 103.8) (end 125.9 103.5) (width 0.6) (layer "B.Cu") (net 3))
-  (segment (start 126 87.2) (end 126 87.1) (width 0.6) (layer "B.Cu") (net 3))
+  (segment (start 84.6 127.2) (end 90 127.2) (width 0.6) (layer "B.Cu") (net 3))
   (segment (start 81.5 76.8) (end 99.4 76.8) (width 0.6) (layer "F.Cu") (net 5))
   (segment (start 72.525 67.825) (end 81.5 76.8) (width 0.6) (layer "F.Cu") (net 5))
@@
   (segment (start 65.3 88.8) (end 72.7 96.2) (width 0.6) (layer "B.Cu") (net 6))
   (segment (start 87.9 122.1) (end 87.9 123.5) (width 0.6) (layer "B.Cu") (net 6))
-  (segment (start 96.1 74.3) (end 103.2 74.3) (width 0.6) (layer "B.Cu") (net 6))
   (segment (start 121.6 106) (end 121.5 106.1) (width 0.6) (layer "B.Cu") (net 6))
-  (segment (start 90.8 69) (end 96.1 74.3) (width 0.6) (layer "B.Cu") (net 6))
+  (segment (start 88.3 69) (end 94.9 75.6) (width 0.6) (layer "B.Cu") (net 6))
+  (segment (start 94.9 75.6) (end 103.1 75.6) (width 0.6) (layer "B.Cu") (net 6))
   (segment (start 72.7 101.8) (end 65.4 109.1) (width 0.6) (layer "B.Cu") (net 6))
   (segment (start 85.9 70.4) (end 87.3 69) (width 0.6) (layer "B.Cu") (net 6))
@@
   (segment (start 105.2 104.8) (end 87.9 122.1) (width 0.6) (layer "B.Cu") (net 6))
   (segment (start 84.45 69.05) (end 84.45 70.55) (width 0.6) (layer "B.Cu") (net 6))
-  (segment (start 103.2 74.3) (end 113.7 84.8) (width 0.6) (layer "B.Cu") (net 6))
-  (segment (start 87.3 69) (end 90.8 69) (width 0.6) (layer "B.Cu") (net 6))
+  (segment (start 103.1 75.6) (end 112.3 84.8) (width 0.6) (layer "B.Cu") (net 6))
+  (segment (start 112.3 84.8) (end 121.6 84.8) (width 0.6) (layer "B.Cu") (net 6))
   (segment (start 121.5 84.9) (end 121.6 84.8) (width 0.6) (layer "B.Cu") (net 6))
   (segment (start 72.7 96.2) (end 72.7 101.8) (width 0.6) (layer "B.Cu") (net 6))
@@
   (segment (start 65.3 81.6) (end 73.4 81.6) (width 0.6) (layer "B.Cu") (net 6))
   (segment (start 121.5 106.1) (end 120.2 104.8) (width 0.6) (layer "B.Cu") (net 6))
-  (segment (start 113.7 84.8) (end 121.6 84.8) (width 0.6) (layer "B.Cu") (net 6))
+  (segment (start 87.3 69) (end 88.3 69) (width 0.6) (layer "B.Cu") (net 6))
   (segment (start 121.6 84.8) (end 121.6 106) (width 0.6) (layer "B.Cu") (net 6))
   (segment (start 65.3 81.6) (end 65.3 88.8) (width 0.6) (layer "B.Cu") (net 6))

Commit message: v2
Parts:
- moved Buck1 23.2 mm to (86.5, 85.8), turned to 0 degrees
- moved H2 19.4 mm to (134.2, 95.5)
- moved H1 5.83 mm to (65.5, 61.2)
- moved H3 4.70 mm to (65.5, 129.7)
- moved J1 1.05 mm to (72.4, 99.1)
Connections:
- J3 pad 2: /D_LAST -> /D_FIRST
- J3 pad 3: /D_FIRST -> /D_LAST
- J4 pad 2: /D_LAST -> /D_FIRST
- J4 pad 3: /D_FIRST -> /D_LAST
- J7 pad 2: /D_LAST -> /D_FIRST
- J7 pad 3: /D_FIRST -> /D_LAST
Routing:
- net +12V: track 200.2 -> 0.00 mm, vias 5 -> 88
- net /D_LAST: track 222.0 -> 204.6 mm, vias 0 -> 10
- net /D_FIRST: track 182.0 -> 194.8 mm, vias 8 -> 0
- net /D_23: track 37.2 -> 45.0 mm, vias 0 -> 2
- net /D_12: track 36.2 -> 43.6 mm, vias 0 -> 2
- net +5V: track 191.7 -> 185.5 mm, vias 2 -> 6
- net /D_45: track 25.9 -> 28.2 mm, vias 0 -> 2
- net /D_34: track 25.9 -> 27.2 mm, vias 0 -> 2
- net /D_56: track 40.3 -> 39.5 mm, vias 0 -> 2
- net GND: vias 19 -> 162
- added copper zone on B.Cu, net +12V
- added copper zone on F.Cu, net +12V
Other:
- board text added: "GND D_LAST D_FIRST +12V"
- board text added: "J3"
- board text removed: "GND D_FIRST D_LAST +12V"

Commit message: v3
Parts:
- added G***: LOGO, --local:logo_kms_small_silkscreen, F.Cu at (96.8, 71.1)
Routing:
- net /D_FIRST: track 194.8 -> 216.7 mm, vias 0 -> 4
- net /D_LAST: track 204.6 -> 208.8 mm, vias 10 -> 8
- net +5V: track 185.5 -> 189.1 mm
- net /D_12: track 43.6 -> 44.9 mm
- net GND: vias 162 -> 159
Other:
- board text added: "Modular rhombus LED panel"
- board text added: "Panel Nr."
- board text added: "V1.0 2024"
- board text added: "makerspace.lt"

Commit message: prieš perdaryma
Parts:
- removed G***: LOGO, --local:logo_kms_small_silkscreen
- added G1: LOGO_KMS, --local:logo_kms_small_silkscreen, F.Cu at (96.3, 70.7)
Routing:
- net /D_FIRST: track 216.7 -> 236.6 mm, vias 4 -> 6
- net /D_LAST: track 208.8 -> 226.0 mm, vias 8 -> 10
- net /D_56: track 39.5 -> 42.8 mm
- net +5V: track 189.1 -> 187.0 mm
- net GND: vias 159 -> 171

Commit message: 2.1
Parts:
- added R1: R, Resistor_SMD:R_0805_2012Metric_Pad1.20x1.40mm_HandSolder, F.Cu at (79.7, 70.7)
- added R2: R, Resistor_SMD:R_0805_2012Metric_Pad1.20x1.40mm_HandSolder, F.Cu at (78.0, 104.5)
- added U1: USBLC6-2SC6, Package_TO_SOT_SMD:SOT-23-6, F.Cu at (76.2, 70.6)
- added U2: USBLC6-2SC6, Package_TO_SOT_SMD:SOT-23-6, F.Cu at (78.1, 100.9)
- moved Buck1 15.5 mm to (89.8, 100.9), turned to 90 degrees
- moved J1 0.55 mm to (71.8, 99.1)
Connections:
- D1 pad 4: /D_FIRST -> Net-(D1-DIN)
- D6 pad 2: /D_LAST -> Net-(D6-DOUT)
Routing:
- net +5V: track 187.0 -> 212.5 mm
- net /D_LAST: track 226.0 -> 245.4 mm
- net /D_FIRST: track 236.6 -> 228.7 mm, vias 6 -> 4
- net Net-(D1-DIN): track 0.00 -> 6.87 mm
- net GND: track 0.00 -> 4.55 mm, vias 171 -> 199
- net /D_56: track 42.8 -> 39.3 mm
- net Net-(D6-DOUT): track 0.00 -> 2.89 mm
- net Net-(R2-Pad2): track 0.00 -> 2.42 mm
- net Net-(R1-Pad1): track 0.00 -> 2.30 mm
- net /D_12: track 45.1 -> 44.1 mm
Other:
- board text added: "+12V D_LAST"
- board text added: "+5V D_FIRST D_LAST GND"
- board text added: "D_FIRST GND"
- board text added: "V1.1 2024"
- board text removed: "+5V D_LAST D_FIRST GND"
- board text removed: "V1.0 2024"
