File: project/makerspace_sign.kicad_sch (KiCad schematic)
At the start: 23 parts, among them J1 Conn_EXT, J2 Conn_E1_M, J3 Conn_E1_F, J4 Conn_OTH_M, J5 Conn_OTH_F, J6 Conn_E2_F, J7 Conn_E2_M

Commit message: v2
Connections:
- net D_FIRST: now also J3.2 (Pin_2), J4.2 (Pin_2), J7.2 (Pin_2); no longer J3.3 (Pin_3), J4.3 (Pin_3), J7.3 (Pin_3)
- net D_LAST: now also J3.3 (Pin_3), J4.3 (Pin_3), J7.3 (Pin_3); no longer J3.2 (Pin_2), J4.2 (Pin_2), J7.2 (Pin_2)
Changed lines of the file:
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@@
     (effects (font (size 1.5 1.5) (thickness 0.3) bold) (justify left bottom))
-  )
-  (label "D_LAST" (at 160.02 140.97 180) (fields_autoplaced)
-    (effects (font (size 1.27 1.27)) (justify right bottom))
   )
   (label "D_LAST" (at 160.02 127 180) (fields_autoplaced)
@@
     (effects (font (size 1.27 1.27)) (justify left bottom))
   )
-  (label "D_FIRST" (at 158.75 104.14 180) (fields_autoplaced)
+  (label "D_LAST" (at 219.71 88.9 180) (fields_autoplaced)
     (effects (font (size 1.27 1.27)) (justify right bottom))
   )
-  (label "D_LAST" (at 219.71 88.9 180) (fields_autoplaced)
+  (label "D_LAST" (at 160.02 143.51 180) (fields_autoplaced)
     (effects (font (size 1.27 1.27)) (justify right bottom))
   )
@@
     (effects (font (size 1.27 1.27)) (justify right bottom))
   )
-  (label "D_FIRST" (at 160.02 143.51 180) (fields_autoplaced)
+  (label "D_45" (at 222.25 43.18 180) (fields_autoplaced)
     (effects (font (size 1.27 1.27)) (justify right bottom))
   )
-  (label "D_45" (at 222.25 43.18 180) (fields_autoplaced)
+  (label "D_LAST" (at 99.06 82.55 180) (fields_autoplaced)
     (effects (font (size 1.27 1.27)) (justify right bottom))
   )
@@
     (effects (font (size 1.27 1.27)) (justify right bottom))
   )
-  (label "D_LAST" (at 99.06 85.09 180) (fields_autoplaced)
+  (label "D_56" (at 248.92 43.18 180) (fields_autoplaced)
     (effects (font (size 1.27 1.27)) (justify right bottom))
   )
-  (label "D_FIRST" (at 99.06 82.55 180) (fields_autoplaced)
-    (effects (font (size 1.27 1.27)) (justify right bottom))
-  )
-  (label "D_LAST" (at 158.75 101.6 180) (fields_autoplaced)
-    (effects (font (size 1.27 1.27)) (justify right bottom))
-  )
-  (label "D_56" (at 248.92 43.18 180) (fields_autoplaced)
+  (label "D_LAST" (at 158.75 104.14 180) (fields_autoplaced)
     (effects (font (size 1.27 1.27)) (justify right bottom))
   )
@@
     (effects (font (size 1.27 1.27)) (justify right bottom))
   )
+  (label "D_FIRST" (at 158.75 101.6 180) (fields_autoplaced)
+    (effects (font (size 1.27 1.27)) (justify right bottom))
+  )
+  (label "D_FIRST" (at 160.02 140.97 180) (fields_autoplaced)
+    (effects (font (size 1.27 1.27)) (justify right bottom))
+  )
   (label "D_12" (at 130.81 43.18 0) (fields_autoplaced)
     (effects (font (size 1.27 1.27)) (justify left bottom))
@@
     (effects (font (size 1.27 1.27)) (justify right bottom))
   )
+  (label "D_FIRST" (at 99.06 85.09 180) (fields_autoplaced)
+    (effects (font (size 1.27 1.27)) (justify right bottom))
+  )

Commit message: v3
Changed lines of the file:
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@@
+    )
+  )
+  (symbol (lib_id "--local:LOGO_KMS") (at 218.44 128.27 0) (unit 1)
+    (in_bom yes) (on_board yes) (dnp no) (fields_autoplaced)
+    (property "Reference" "#G1" (at 218.44 114.3423 0)
+      (effects (font (size 1.27 1.27)) hide)
+    )
+    (property "Value" "LOGO_KMS" (at 218.44 142.1977 0)
+      (effects (font (size 1.27 1.27)) hide)
+    )
+    (property "Footprint" "--local:logo_kms_small_silkscreen" (at 218.44 128.27 0)
+      (effects (font (size 1.27 1.27)) hide)
+    )
+    (property "Datasheet" "" (at 218.44 128.27 0)
+      (effects (font (size 1.27 1.27)) hide)
+    )
+    (instances
+      (project "makerspace_sign"
+        (path "/671df12e-dade-4f44-8399-d2645e1bafe3"
+          (reference "#G1") (unit 1)
+        )
+      )
     )
   )

Commit message: prieš perdaryma
Parts:
- added G1: LOGO_KMS, --local:logo_kms_small_silkscreen, symbol --local:LOGO_KMS
Changed lines of the file:
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@@
+    )
+  )
+  (symbol (lib_id "--local:LOGO_KMS") (at 223.52 130.81 0) (unit 1)
+    (in_bom yes) (on_board yes) (dnp no) (fields_autoplaced)
+    (property "Reference" "G1" (at 223.52 116.8823 0)
+      (effects (font (size 1.27 1.27)) hide)
+    )
+    (property "Value" "LOGO_KMS" (at 223.52 144.7377 0)
+      (effects (font (size 1.27 1.27)) hide)
+    )
+    (property "Footprint" "--local:logo_kms_small_silkscreen" (at 223.52 130.81 0)
+      (effects (font (size 1.27 1.27)) hide)
+    )
+    (property "Datasheet" "" (at 223.52 130.81 0)
+      (effects (font (size 1.27 1.27)) hide)
+    )
+    (instances
+      (project "makerspace_sign"
+        (path "/671df12e-dade-4f44-8399-d2645e1bafe3"
+          (reference "G1") (unit 1)
+        )
+      )
     )
   )
@@
         )
       )
-    )
-  )
-  (symbol (lib_id "--local:LOGO_KMS") (at 218.44 128.27 0) (unit 1)
-    (in_bom yes) (on_board yes) (dnp no) (fields_autoplaced)
-    (property "Reference" "#G1" (at 218.44 114.3423 0)
-      (effects (font (size 1.27 1.27)) hide)
-    )
-    (property "Value" "LOGO_KMS" (at 218.44 142.1977 0)
-      (effects (font (size 1.27 1.27)) hide)
-    )
-    (property "Footprint" "--local:logo_kms_small_silkscreen" (at 218.44 128.27 0)
-      (effects (font (size 1.27 1.27)) hide)
-    )
-    (property "Datasheet" "" (at 218.44 128.27 0)
-      (effects (font (size 1.27 1.27)) hide)
-    )
-    (instances
-      (project "makerspace_sign"
-        (path "/671df12e-dade-4f44-8399-d2645e1bafe3"
-          (reference "#G1") (unit 1)
-        )
-      )

Commit message: 2.1
Parts:
- added R1, R2: R, Resistor_SMD:R_0805_2012Metric_Pad1.20x1.40mm_HandSolder, symbol Device:R
- added U1 (x2): USBLC6-2SC6, Package_TO_SOT_SMD:SOT-23-6, symbol Power_Protection:USBLC6-2SC6
Connections:
- net +5V: now also U1.5 (VBUS), U1.5 (VBUS)
- net D_FIRST: now also R1.2; no longer D1.4 (DIN)
- net D_LAST: now also R2.1; no longer D6.2 (DOUT)
- net GND: now also U1.2 (GND), U1.2 (GND)
- new net: R1.1, U1.3 (I/O2)
- new net: D1.4 (DIN), U1.4 (I/O2)
- new net: R2.2, U1.6 (I/O1)
- new net: D6.2 (DOUT), U1.1 (I/O1)
- no-connect marks 1 -> 5
Other:
- moved on the sheet: Buck1, C1, C2, C3, C4, C5, C6, D1, D2, D3, D4, D5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
